File: hardware/TrinketTrigger.sch (EAGLE design)
At the start: 11 parts, among them IC1 7805L, J1 THONKICONNNEW, J2 THONKICONNNEW

Commit message: added sch pdf
Other:
- note added: "2020 @todbot / Tod E. Kurt"
Changed lines of the file:
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@@
 <?xml version="1.0" encoding="utf-8"?>
 <!DOCTYPE eagle SYSTEM "eagle.dtd">
-<eagle version="9.6.1">
+<eagle version="9.6.2">
 <drawing>
 <settings>
-<setting alwaysvectorfont="no"/>
+<setting alwaysvectorfont="yes"/>
 <setting verticaltext="up"/>
 </settings>
@@
 <part name="S1" library="SparkFun-Switches" library_urn="urn:adsk.eagle:library:535" deviceset="MOMENTARY-SWITCH-SPST" device="-PTH-6.0MM" package3d_urn="urn:adsk.eagle:package:40163/1"/>
 <part name="GND7" library="supply1" library_urn="urn:adsk.eagle:library:371" deviceset="GND" device=""/>
-<part name="FRAME1" library="frames" library_urn="urn:adsk.eagle:library:229" deviceset="A4L-LOC" device=""/>
+<part name="FRAME1" library="frames" library_urn="urn:adsk.eagle:library:229" deviceset="A4L-LOC" device="" value="TrinketTrigger @todbot"/>
 </parts>
 <sheets>
 <sheet>
 <plain>
+<text x="218.44" y="20.32" size="1.778" layer="94" ratio="12">2020 @todbot / Tod E. Kurt</text>
 </plain>
 <instances>
